File: LVDS_serialization.kicad_sch (KiCad schematic)
At the start: 23 parts, among them IC3 DS90LV048ATM_NOPB, IC4 DS90LV048ATM_NOPB, IC5 DS90LV048ATM_NOPB, IC6 DS90LV048ATM_NOPB, IC7 DS90LV048ATM_NOPB

Commit message: Corrected LVDS
Parts:
- removed IC6, IC7: DS90LV048ATM_NOPB, SOIC127P600X175-16N, symbol SamacSys_Parts:DS90LV048ATM_NOPB
- removed RLVDS11, RLVDS12, RLVDS13, RLVDS14, RLVDS15, RLVDS16, RLVDS17, RLVDS18: 100, symbol Device:R_Small
Connections:
- net DOUT10 is gone; now on net DOUT6: IC4.10 (ROUT4)
- net DOUT12 is gone; now on net DOUTCTR: IC3.11 (ROUT3)
- net DOUT13 is gone; now on net DOUT3: IC5.15 (ROUT1)
- net DOUT15 is gone; now on net DOUT4: IC3.10 (ROUT4)
- net LVDS_10N is gone; now on net LVDS_6N: IC4.8 (RIN4-), RLVDS8.2
- net LVDS_10P is gone; now on net LVDS_6P: IC4.7 (RIN4+), RLVDS8.1
- net LVDS_12N is gone; now on net LVDS_CTRN: IC3.5 (RIN3-), RLVDS3.1
- net LVDS_12P is gone; now on net LVDS_CTRP: IC3.6 (RIN3+), RLVDS3.2
- net LVDS_13N is gone; now on net LVDS_3N: IC5.1 (RIN1-), RLVDS9.1
- net LVDS_13P is gone; now on net LVDS_3P: IC5.2 (RIN1+), RLVDS9.2
- net LVDS_15N is gone; now on net LVDS_4N: IC3.8 (RIN4-), RLVDS4.2
- net LVDS_15P is gone; now on net LVDS_4P: IC3.7 (RIN4+), RLVDS4.1
- net DOUT1: now also IC4.11 (ROUT3); no longer IC5.11 (ROUT3)
- net DOUT4: no longer IC4.14 (ROUT2)
- net DOUT6: no longer IC5.10 (ROUT4)
- net DOUT7: now also IC4.15 (ROUT1); no longer IC4.11 (ROUT3)
- net DOUT8: now also IC5.14 (ROUT2)
- net DOUTCLK: now also IC4.14 (ROUT2); no longer IC5.14 (ROUT2)
- net DOUTCTR: no longer IC4.15 (ROUT1)
- net LVDS_1N: now also IC4.5 (RIN3-), RLVDS7.1; no longer IC5.5 (RIN3-)
- net LVDS_1P: now also IC4.6 (RIN3+), RLVDS7.2; no longer IC5.6 (RIN3+)
- net LVDS_4N: no longer IC4.4 (RIN2-), RLVDS6.2
- net LVDS_4P: no longer IC4.3 (RIN2+), RLVDS6.1
- net LVDS_6N: no longer IC5.8 (RIN4-)
- net LVDS_6P: no longer IC5.7 (RIN4+)
- net LVDS_7N: now also IC4.1 (RIN1-), RLVDS5.1; no longer IC4.5 (RIN3-), RLVDS7.1
- net LVDS_7P: now also IC4.2 (RIN1+), RLVDS5.2; no longer IC4.6 (RIN3+), RLVDS7.2
- net LVDS_8N: now also IC5.4 (RIN2-), RLVDS10.2
- net LVDS_8P: now also IC5.3 (RIN2+), RLVDS10.1
- net LVDS_CLKN: now also IC4.4 (RIN2-), RLVDS6.2; no longer IC5.4 (RIN2-), RLVDS10.2
- net LVDS_CLKP: now also IC4.3 (RIN2+), RLVDS6.1; no longer IC5.3 (RIN2+), RLVDS10.1
- net LVDS_CTRN: no longer IC4.1 (RIN1-), RLVDS5.1
- net LVDS_CTRP: no longer IC4.2 (RIN1+), RLVDS5.2
- no-connect marks 9 -> 5

Commit message: Added lots more connections
Parts:
- added C17, C20, C22: 0.1uF, symbol Device:C_Polarized
- added C18, C19, C21: 1nF, symbol Device:C_Polarized
Connections:
- net +3V3: now also C17.1, C18.1, C19.1, C20.1, C21.1, C22.1
- net GNDSIG renamed GND
- net GND: now also C17.2, C18.2, C19.2, C20.2, C21.2, C22.2
