File: lvds.kicad_sch (KiCad schematic)
At the start: 19 parts, among them IC3 DS90LV048ATM_NOPB, IC4 DS90LV048ATM_NOPB, IC5 DS90LV048ATM_NOPB

Commit message: One gnd to rule them all; PCB border (90 mm x 90 mm)
Connections:
- net GNDSIG_A renamed GND

Commit message: 3v3 Regulator routed; zones for 3v3 and gnd
Parts:
- IC3, IC4, IC5: footprint SOIC127P600X175-16N -> SamacSys_Parts:SOIC127P600X175-16N
Changed lines of the file:
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@@
+	)
+	(symbol
+		(lib_id "SamacSys_Parts:DS90LV048ATM_NOPB")
+		(at 114.3 125.73 0)
+		(unit 1)
+		(exclude_from_sim no)
+		(in_bom yes)
+		(on_board yes)
+		(dnp no)
+		(fields_autoplaced yes)
+		(property "Reference" "IC5"
+			(at 130.81 118.11 0)
+			(effects
+				(font
+					(size 1.27 1.27)
+				)
+			)
+		)
+		(property "Value" "DS90LV048ATM_NOPB"
+			(at 130.81 120.65 0)
+			(effects
+				(font
+					(size 1.27 1.27)
+				)
+			)
+		)
+		(property "Footprint" "SamacSys_Parts:SOIC127P600X175-16N"
+			(at 143.51 220.65 0)
+			(effects
+				(font
+					(size 1.27 1.27)
+				)
+				(justify left top)
+				(hide yes)
+			)
+		)
+		(property "Datasheet" "http://www.ti.com/lit/ds/symlink/ds90lv048a.pdf"
+			(at 143.51 320.65 0)
+			(effects
+				(font
+					(size 1.27 1.27)
+				)
+				(justify left top)
+				(hide yes)
+			)
+		)
+		(property "Description" "400 Mbps LVDS Quad High Speed Differential Receiver"
+			(at 114.3 125.73 0)
+			(effects
+				(font
+					(size 1.27 1.27)
+				)
+				(hide yes)
+			)
+		)
+		(property "Height" "1.75"
+			(at 143.51 520.65 0)
+			(effects
+				(font
+					(size 1.27 1.27)
+				)
+				(justify left top)
+				(hide yes)
+			)
+		)
+		(property "Manufacturer_Name" "Texas Instruments"
+			(at 143.51 620.65 0)
+			(effects
+				(font
+					(size 1.27 1.27)
+				)
+				(justify left top)
+				(hide yes)
+			)
+		)
+		(property "Manufacturer_Part_Number" "DS90LV048ATM/NOPB"
+			(at 143.51 720.65 0)
+			(effects
+				(font
+					(size 1.27 1.27)
+				)
+				(justify left top)
+				(hide yes)
+			)
+		)
+		(property "Arrow Part Number" "DS90LV048ATM/NOPB"
+			(at 143.51 820.65 0)
+			(effects
+				(font
+					(size 1.27 1.27)
+				)
+				(justify left top)
+				(hide yes)
+			)
+		)
+		(property "Arrow Price/Stock" "null?region=nac"
+			(at 143.51 920.65 0)
+			(effects
+				(font
+					(size 1.27 1.27)
+				)
+				(justify left top)
+				(hide yes)
+			)
+		)
+		(pin "7"
+		)
+		(pin "3"
+		)
+		(pin "4"
+		)
+		(pin "12"
+		)
+		(pin "15"
+		)
+		(pin "1"
+		)
+		(pin "11"
+		)
+		(pin "14"
+		)
+		(pin "13"
+		)
+		(pin "5"
+		)
+		(pin "10"
+		)
+		(pin "8"
+		)
+		(pin "2"
+		)
+		(pin "16"
+		)
+		(pin "9"
+		)
+		(pin "6"
+		)
+		(instances
+			(project "S25-26"
+				(path "/6f4563ef-8a79-4567-b913-33c6dfb42b56/10aa7ffc-4759-4dd0-b397-4be5b97e2346"
+					(reference "IC5")
+					(unit 1)
+				)
+			)
+		)
 	)
 	(symbol
@@
 	(symbol
 		(lib_id "SamacSys_Parts:DS90LV048ATM_NOPB")
-		(at 114.3 125.73 0)
+		(at 114.3 86.36 0)
 		(unit 1)
 		(exclude_from_sim no)
@@
 		(dnp no)
 		(fields_autoplaced yes)
-		(property "Reference" "IC5"
-			(at 130.81 118.11 0)
+		(property "Reference" "IC4"
+			(at 130.81 78.74 0)
 			(effects
 				(font
@@
 		)
 		(property "Value" "DS90LV048ATM_NOPB"
-			(at 130.81 120.65 0)
-			(effects
-				(font
-					(size 1.27 1.27)
-				)
-			)
-		)
-		(property "Footprint" "SOIC127P600X175-16N"
-			(at 143.51 220.65 0)
+			(at 130.81 81.28 0)
+			(effects
+				(font
+					(size 1.27 1.27)
+				)
+			)
+		)
+		(property "Footprint" "SamacSys_Parts:SOIC127P600X175-16N"
+			(at 143.51 181.28 0)
 			(effects
 				(font
@@
 		)
 		(property "Datasheet" "http://www.ti.com/lit/ds/symlink/ds90lv048a.pdf"
-			(at 143.51 320.65 0)
+			(at 143.51 281.28 0)
 			(effects
 				(font
@@
 		)
 		(property "Description" "400 Mbps LVDS Quad High Speed Differential Receiver"
-			(at 114.3 125.73 0)
+			(at 114.3 86.36 0)
 			(effects
 				(font
@@
 		)
 		(property "Height" "1.75"
-			(at 143.51 520.65 0)
+			(at 143.51 481.28 0)
 			(effects
 				(font
@@
 		)
 		(property "Manufacturer_Name" "Texas Instruments"
-			(at 143.51 620.65 0)
+			(at 143.51 581.28 0)
 			(effects
 				(font
@@
 		)
 		(property "Manufacturer_Part_Number" "DS90LV048ATM/NOPB"
-			(at 143.51 720.65 0)
+			(at 143.51 681.28 0)
 			(effects
 				(font
@@
 		)
 		(property "Arrow Part Number" "DS90LV048ATM/NOPB"
-			(at 143.51 820.65 0)
+			(at 143.51 781.28 0)
 			(effects
 				(font
@@
 		)
 		(property "Arrow Price/Stock" "null?region=nac"
-			(at 143.51 920.65 0)
+			(at 143.51 881.28 0)
 			(effects
 				(font
@@
 			(project "S25-26"
 				(path "/6f4563ef-8a79-4567-b913-33c6dfb42b56/10aa7ffc-4759-4dd0-b397-4be5b97e2346"
-					(reference "IC5")
+					(reference "IC4")
 					(unit 1)
 				)
@@
 	)
 	(symbol
-		(lib_id "SamacSys_Parts:DS90LV048ATM_NOPB")
-		(at 114.3 86.36 0)
-		(unit 1)
-		(exclude_from_sim no)
-		(in_bom yes)
-		(on_board yes)
-		(dnp no)
-		(fields_autoplaced yes)
-		(property "Reference" "IC4"
-			(at 130.81 78.74 0)
-			(effects
-				(font
-					(size 1.27 1.27)
-				)
-			)
-		)
-		(property "Value" "DS90LV048ATM_NOPB"
-			(at 130.81 81.28 0)
-			(effects
-				(font
-					(size 1.27 1.27)
-				)
-			)
-		)
-		(property "Footprint" "SOIC127P600X175-16N"
-			(at 143.51 181.28 0)
-			(effects
-				(font
-					(size 1.27 1.27)
-				)
-				(justify left top)
-				(hide yes)
-			)
-		)
-		(property "Datasheet" "http://www.ti.com/lit/ds/symlink/ds90lv048a.pdf"
-			(at 143.51 281.28 0)
-			(effects
-				(font
-					(size 1.27 1.27)
-				)
-				(justify left top)
-				(hide yes)
-			)
-		)
-		(property "Description" "400 Mbps LVDS Quad High Speed Differential Receiver"
-			(at 114.3 86.36 0)
-			(effects
-				(font
-					(size 1.27 1.27)
-				)
-				(hide yes)
-			)
-		)
-		(property "Height" "1.75"
-			(at 143.51 481.28 0)
-			(effects
-				(font
-					(size 1.27 1.27)
-				)
-				(justify left top)
-				(hide yes)
-			)
-		)
-		(property "Manufacturer_Name" "Texas Instruments"
-			(at 143.51 581.28 0)
-			(effects
-				(font
-					(size 1.27 1.27)
-				)
-				(justify left top)
-				(hide yes)
-			)
-		)
-		(property "Manufacturer_Part_Number" "DS90LV048ATM/NOPB"
-			(at 143.51 681.28 0)
-			(effects
-				(font
-					(size 1.27 1.27)
-				)
-				(justify left top)
-				(hide yes)
-			)
-		)
-		(property "Arrow Part Number" "DS90LV048ATM/NOPB"
-			(at 143.51 781.28 0)
-			(effects
-				(font
-					(size 1.27 1.27)
-				)
-				(justify left top)
-				(hide yes)
-			)
-		)
-		(property "Arrow Price/Stock" "null?region=nac"
-			(at 143.51 881.28 0)
-			(effects
-				(font
-					(size 1.27 1.27)
-				)
-				(justify left top)
-				(hide yes)
-			)
-		)
-		(pin "7"
-		)
-		(pin "3"
-		)
-		(pin "4"
-		)
-		(pin "12"
-		)
-		(pin "15"
-		)
-		(pin "1"
-		)
-		(pin "11"
-		)
-		(pin "14"
-		)
-		(pin "13"
-		)
-		(pin "5"
-		)
-		(pin "10"
-		)
-		(pin "8"
-		)
-		(pin "2"
-		)
-		(pin "16"
-		)
-		(pin "9"
-		)
-		(pin "6"
-		)
-		(instances
-			(project "S25-26"
-				(path "/6f4563ef-8a79-4567-b913-33c6dfb42b56/10aa7ffc-4759-4dd0-b397-4be5b97e2346"
-					(reference "IC4")
-					(unit 1)
-				)
-			)
-		)
-	)
-	(symbol
 		(lib_id "Device:R_Small")
 		(at 105.41 59.69 0)
@@
 			)
 		)
-		(property "Footprint" "SOIC127P600X175-16N"
+		(property "Footprint" "SamacSys_Parts:SOIC127P600X175-16N"
 			(at 143.51 141.91 0)
 			(effects

Commit message: Schematic - Component Specifics
Fixed floating connections.
Added parameters, footprints, Mouser part numbers, and Mouser links to all symbols, including discrete components and ICs.
The following symbols do not have Mouser part numbers or Mouser links:
CMOS Sensor (not required)
RJ45 Connector
JTAG Connector
DC Barrel Jack
Parts:
- removed C17, C18, C19: 1nF, symbol Device:C_Polarized
- added C17, C18, C19: 1nF, Capacitor_SMD:C_0603_1608Metric, symbol Device:C_Small
- C20, C21, C22: footprint (none) -> Capacitor_SMD:C_0805_2012Metric; Dielectric (none) -> TANT; Mouser Part Number (none) -> 581-TAJR104K020R; Mouser Price/Stock (none) -> https://www.mouser.com/ProductDetail/KYOCERA-AVX/TAJR104K02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; Tolerance (none) -> 10%; Voltage Rating (none) -> 20V
- IC3, IC4, IC5: Arrow Part Number DS90LV048ATM/NOPB -> (none); Arrow Price/Stock null?region=nac -> (none); Mosuer Price/Stock (none) -> https://www.mouser.com/ProductDetail/Texas-Instruments/DS90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; Mouser Part Number (none) -> :926-DS90LV048ATMNOPB
- RLVDS1, RLVDS10, RLVDS2, RLVDS3, RLVDS4, RLVDS5, RLVDS6, RLVDS7, RLVDS8, RLVDS9: footprint (none) -> Resistor_SMD:R_0603_1608Metric; Mouser Part Number (none) -> 71-CRCW0603100RFKEAH; Mouser Price/Stock (none) -> https://www.mouser.com/ProductDetail/Vishay-Dale/CRCW060310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; Power Rating (none) -> 0.33W; Tolerance (none) -> 1%
Connections:
- net +3V3: now also C17.1, C18.1, C19.1
- net GND: now also C17.2, C18.2, C19.2
- net LVDS_CH03_N: now also RLVDS7.1; no longer RLVDS7.2
- net LVDS_CH03_P: now also RLVDS7.2; no longer RLVDS7.1
- net LVDS_CH07_N: now also RLVDS3.1; no longer RLVDS3.2
- net LVDS_CH07_P: now also RLVDS3.2; no longer RLVDS3.1
- net LVDS_CH09_N: now also RLVDS8.2; no longer RLVDS8.1
- net LVDS_CH09_P: now also RLVDS8.1; no longer RLVDS8.2
- net LVDS_CH13_N: now also RLVDS4.2; no longer RLVDS4.1
- net LVDS_CH13_P: now also RLVDS4.1; no longer RLVDS4.2
- net LVDS_CTR_OUT_N: now also RLVDS10.2; no longer RLVDS10.1
- net LVDS_CTR_OUT_P: now also RLVDS10.1; no longer RLVDS10.2

Commit message: Some small changes for BOM
Parts:
- IC3, IC4, IC5: Mosuer Price/Stock https://www.mouser.com/ProductDetail/Texas-Instruments/DS90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 -> (none); Mouser Price/Stock (none) -> https://www.mouser.com/ProductDetail/Texas-Instruments/DS90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
Changed lines of the file:
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@@
 			)
 		)
-		(property "Mosuer Price/Stock" "https://www.mouser.com/ProductDetail/Texas-Instruments/DS90LV048ATM-NOPB?qs=X1J7HmVL2ZGZM9KQD2xuIA%3D%3D"
+		(property "Mouser Price/Stock" "https://www.mouser.com/ProductDetail/Texas-Instruments/DS90LV048ATM-NOPB?qs=X1J7HmVL2ZGZM9KQD2xuIA%3D%3D"
 			(at 143.51 881.28 0)
 			(effects
@@
 			)
 		)
-		(property "Mosuer Price/Stock" "https://www.mouser.com/ProductDetail/Texas-Instruments/DS90LV048ATM-NOPB?qs=X1J7HmVL2ZGZM9KQD2xuIA%3D%3D"
+		(property "Mouser Price/Stock" "https://www.mouser.com/ProductDetail/Texas-Instruments/DS90LV048ATM-NOPB?qs=X1J7HmVL2ZGZM9KQD2xuIA%3D%3D"
 			(at 143.51 920.65 0)
 			(effects
@@
 			)
 		)
-		(property "Mosuer Price/Stock" "https://www.mouser.com/ProductDetail/Texas-Instruments/DS90LV048ATM-NOPB?qs=X1J7HmVL2ZGZM9KQD2xuIA%3D%3D"
+		(property "Mouser Price/Stock" "https://www.mouser.com/ProductDetail/Texas-Instruments/DS90LV048ATM-NOPB?qs=X1J7HmVL2ZGZM9KQD2xuIA%3D%3D"
 			(at 143.51 841.91 0)
 			(effects

Commit message: Ethernet Transceiver
Parts:
- renumbered C17 to C65, C18 to C66, C19 to C67, C20 to C68, C21 to C69, C22 to C70, IC5 to IC10, IC3 to IC8, IC4 to IC9, RLVDS9 to RLVDS10, RLVDS10 to RLVDS11, RLVDS1 to RLVDS2, RLVDS2 to RLVDS3, RLVDS3 to RLVDS4, RLVDS4 to RLVDS5, RLVDS5 to RLVDS6, RLVDS6 to RLVDS7, RLVDS7 to RLVDS8, RLVDS8 to RLVDS9

Commit message: Lots of PCB changes, some small parts changes
Updated parts footprints from those found in MDE Lab. Some parameters may be incorrect, but all footprints should be correct
Drew most of PCB. CMOS SPI still needs connection. Decoupling caps on MCU still need connection. Power and ground needs to be analyzed, and some components may not have power or ground connected.
Connections:
- net CMOS_CH01: now also IC10.15 (ROUT1); no longer IC9.15 (ROUT1)
- net CMOS_CH03: now also IC9.10 (ROUT4); no longer IC9.11 (ROUT3)
- net CMOS_CH05: now also IC9.11 (ROUT3); no longer IC8.15 (ROUT1)
- net CMOS_CH07: now also IC9.14 (ROUT2); no longer IC8.11 (ROUT3)
- net CMOS_CH09: now also IC9.15 (ROUT1); no longer IC9.10 (ROUT4)
- net CMOS_CH11: now also IC8.10 (ROUT4); no longer IC9.14 (ROUT2)
- net CMOS_CH13: now also IC8.11 (ROUT3); no longer IC8.10 (ROUT4)
- net CMOS_CLK_OUT: now also IC8.15 (ROUT1); no longer IC10.10 (ROUT4)
- net CMOS_CTR_OUT: now also IC10.14 (ROUT2); no longer IC10.15 (ROUT1)
- net LVDS_CH01_N: now also IC10.1 (RIN1-), RLVDS10.1; no longer IC9.1 (RIN1-), RLVDS6.1
- net LVDS_CH01_P: now also IC10.2 (RIN1+), RLVDS10.2; no longer IC9.2 (RIN1+), RLVDS6.2
- net LVDS_CH03_N: now also IC9.8 (RIN4-), RLVDS9.2; no longer IC9.5 (RIN3-), RLVDS8.1
- net LVDS_CH03_P: now also IC9.7 (RIN4+), RLVDS9.1; no longer IC9.6 (RIN3+), RLVDS8.2
- net LVDS_CH05_N: now also IC9.5 (RIN3-), RLVDS8.1; no longer IC8.1 (RIN1-), RLVDS2.1
- net LVDS_CH05_P: now also IC9.6 (RIN3+), RLVDS8.2; no longer IC8.2 (RIN1+), RLVDS2.2
- net LVDS_CH07_N: now also IC9.4 (RIN2-), RLVDS7.2; no longer IC8.5 (RIN3-), RLVDS4.1
- net LVDS_CH07_P: now also IC9.3 (RIN2+), RLVDS7.1; no longer IC8.6 (RIN3+), RLVDS4.2
- net LVDS_CH09_N: now also IC9.1 (RIN1-), RLVDS6.1; no longer IC9.8 (RIN4-), RLVDS9.2
- net LVDS_CH09_P: now also IC9.2 (RIN1+), RLVDS6.2; no longer IC9.7 (RIN4+), RLVDS9.1
- net LVDS_CH11_N: now also IC8.8 (RIN4-), RLVDS5.2; no longer IC9.4 (RIN2-), RLVDS7.2
- net LVDS_CH11_P: now also IC8.7 (RIN4+), RLVDS5.1; no longer IC9.3 (RIN2+), RLVDS7.1
- net LVDS_CH13_N: now also IC8.5 (RIN3-), RLVDS4.1; no longer IC8.8 (RIN4-), RLVDS5.2
- net LVDS_CH13_P: now also IC8.6 (RIN3+), RLVDS4.2; no longer IC8.7 (RIN4+), RLVDS5.1
- net LVDS_CLK_OUT_N: now also IC8.1 (RIN1-), RLVDS2.1; no longer IC10.1 (RIN1-), RLVDS10.1
- net LVDS_CLK_OUT_P: now also IC8.2 (RIN1+), RLVDS2.2; no longer IC10.2 (RIN1+), RLVDS10.2
- net LVDS_CTR_OUT_N: now also IC10.4 (RIN2-); no longer IC10.8 (RIN4-)
- net LVDS_CTR_OUT_P: now also IC10.3 (RIN2+); no longer IC10.7 (RIN4+)
- no-connect marks 0 -> 2
Other:
- moved on the sheet: RLVDS11
